Commit message: wip

File: eli_cs_robot_description/urdf/cs_macro.xacro (robot description, xacro)
@@ -202,9 +202,15 @@
       <xacro:build_inertial mass="${wrist_3_mass}" cog="${prop_wrist_3_cog}" inertia="${prop_wrist_3_inertia}"/>
     </link>
-    <!-- base_joint fixes base_link to the environment -->
+    <link name="fts_link" />
+    <joint name="fts_link_joint" type="fixed">
+      <parent link="${parent}" />
+      <child link="fts_link" />
+      <origin xyz="0.0 0 0.0" rpy="3.14 0 3.14" />
+    </joint>
+     <!-- base_joint fixes base_link to the environment -->
     <joint name="${tf_prefix}base_joint" type="fixed">
-      <xacro:insert_block name="origin" />
-      <parent link="${parent}" />
+      <parent link="fts_link" />
       <child link="${tf_prefix}base_link" />
+      <origin xyz="0.0 0 0.0" rpy="-3.14 0 -3.14" />
     </joint>
     <!-- joints - main serial chain -->
